File: boardConsolePCB/boardConsolePCB.kicad_sch (KiCad schematic)
At the start: 132 parts, among them J1 to HV cable, J2 SMA F, J3 PROG, J4 BUTTONS, J5 PWR, J6 FUEL/TRIM, J7 PRG_UART, Q1 BC548, Q2 IRML0030TR, Q3 IRML0030TR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

Commit message: add GDT
Parts:
- added GD1: CG90L, boardConsoleLib:CG90L, symbol Device:GDT_2Pin
Connections:
- net GND: now also GD1.1
- net at D2.1 (K), R3.2, R34.1: now also GD1.3
Other:
- moved on the sheet: C2, C3, J1, R16, R17, R3
